Commit message: updated battery plugin

File: tribot_description/urdf/tribot.urdf (robot description, URDF)
Before this commit: robot tribot, 4 links, 3 joints
Links:
- added link battery_link, mass 0.001
Joints:
- added joint battery_joint: type revolute, parent base_link, child battery_link, origin xyz=0 0 0 rpy=0 0 0, axis 1 0 0, limit lower=0 upper=0 effort=0 velocity=0

Commit message: fixed gazebo callback

File: tribot_description/urdf/tribot.urdf (robot description, URDF)
Before this commit: robot tribot, 5 links, 4 joints
Joints:
- joint battery_joint: axis 1 0 0 -> (none); limit lower=0 upper=0 effort=0 velocity=0 -> (none); origin xyz=0 0 0 rpy=0 0 0 -> xyz=0 0 0.01; type revolute -> fixed

Commit message: rviz2 for fake node

File: tribot_description/urdf/tribot.urdf (robot description, URDF)
Before this commit: robot tribot, 5 links, 4 joints
Links:
- removed link battery_link
Joints:
- removed joint battery_joint

Commit message: added laser sensor

File: tribot_description/urdf/tribot.urdf (robot description, URDF)
Before this commit: robot tribot, 5 links, 4 joints
Links:
- added link laser_link; collision cylinder length=0.1 radius=0.05; visual cylinder length=0.1 radius=0.05
Joints:
- added joint joint_sensor_laser: type fixed, parent base_link, child laser_link, origin xyz=0.15 0 0.05 rpy=0 0 0
